File: hardware/oled-128x64.kicad_pcb (KiCad board)
At the start: 2 copper layers, 40 x 40 mm, 27 parts, among them P1 CON-SENSOR, U1 M24C64, U2 SNGL_NAND, U3 OLED013, U4 DRILL, U5 DRILL, U6 DRILL, U7 DRILL

Commit message: oled version 1.1 * add connector for display
Parts:
- C1, C10, C11, C2, C4, C6, C8, R1: footprint kicad-libraries:0603 -> kicad-libraries:0603E
- G***: footprint kicad-libraries:Logo_31x31m -> kicad-libraries:Logo_31x31
- U3: footprint kicad-libraries:OLED013 -> kicad-libraries:ER-CON30HT-1
- moved G*** 17.9 mm to (166.8, 144.3)
- moved VAL 11.1 mm to (166.8, 137.8)
- moved C3 4.57 mm to (156.2, 140.5), turned to 0 degrees
- moved C5 4.43 mm to (159.9, 140.5), turned to 180 degrees
- moved C10 4.41 mm to (161.8, 143.1), turned to 90 degrees
- moved C8 4.17 mm to (160.3, 143.1)
- moved C6 4.13 mm to (158.2, 143.1), turned to 270 degrees
- moved C4 3.54 mm to (156.5, 143.1), turned to 270 degrees
- moved R1 3.11 mm to (149.7, 143.7)
- moved C7 3.05 mm to (149.0, 142.1)
- moved C9 3.01 mm to (145.5, 142.1)
- moved U3 2.90 mm to (154.1, 146.6), turned to 0 degrees
- moved C11 2.72 mm to (145.4, 143.7)
Routing:
- net GND: track 53.0 -> 37.1 mm, vias 29 -> 27
- net Net-(RP1-Pad8): track 12.3 -> 9.01 mm
- net Net-(RP1-Pad7): track 12.1 -> 8.93 mm
- net Net-(RP1-Pad6): track 11.5 -> 8.64 mm
- net Net-(RP1-Pad5): track 11.6 -> 8.76 mm
- net Net-(C10-Pad1): track 5.99 -> 3.42 mm
- net Net-(U2-Pad4): track 20.0 -> 17.4 mm
- net 3V3: track 82.7 -> 80.6 mm
- net Net-(C10-Pad2): track 4.10 -> 5.92 mm
- net Net-(C8-Pad1): track 5.59 -> 4.21 mm
- net Net-(C8-Pad2): track 3.70 -> 2.51 mm
- net Net-(R1-Pad1): track 3.39 -> 2.70 mm
Other:
- board text added: "OLED 128x64 1.1"
- board text removed: "OLED 128x64 1.0"

Commit message: Add 3d information (tbc)
Parts:
- C1, C10, C11, C2, C4, C6, C8: footprint kicad-libraries:0603E -> kicad-libraries:C0603E
- C3, C5, C7, C9: footprint kicad-libraries:0805 -> kicad-libraries:C0805
- R1: footprint kicad-libraries:0603E -> kicad-libraries:R0603E
Connections:
- P1 pad 1: (no net) -> Net-(P1-Pad1)
- U1 pad 7: (no net) -> Net-(U1-Pad7)
- U3 pad 20: (no net) -> Net-(U3-Pad20)
- U3 pad 7: (no net) -> Net-(U3-Pad7)
